Commit message: removed gripper

File: interbotix_ros_xsarms/interbotix_xsarm_descriptions/urdf/mobile_wx250s.urdf.xacro (robot description, xacro)
@@ -83,5 +83,5 @@
   <joint name="shoulder" type="revolute">
     <axis xyz="0 1 0"/>
-    <limit effort="20" lower="${radians(-108)}" upper="${radians(114)}" velocity="${pi}"/>
+    <limit effort="2" lower="${radians(-108)}" upper="${radians(114)}" velocity="${pi}"/>
     <origin rpy="0 0 0" xyz="0 0 0.03865"/>
     <parent link="$(arg robot_name)/shoulder_link"/>
@@ -278,5 +278,5 @@
     </inertial>
   </link>
-  <joint name="gripper" type="continuous">
+  <!-- <joint name="gripper" type="continuous">
     <axis xyz="1 0 0"/>
     <limit effort="1" velocity="${pi}"/>
@@ -314,7 +314,7 @@
       <inertia ixx="0.0000005923" iyy="0.0000011156" izz="0.0000005743" ixy="0.0000000000" ixz="0.0000003195" iyz="-0.0000000004" />
     </inertial>
-  </link>
+  </link> -->
   <!-- If the AR tag is being used, then add the AR tag mount -->
-  <xacro:if value="$(arg show_ar_tag)">
+  <!-- <xacro:if value="$(arg show_ar_tag)">
     <joint name="ar_tag" type="fixed">
       <axis xyz="0 0 0"/>
@@ -343,7 +343,7 @@
       </inertial>
     </link>
-  </xacro:if>
+  </xacro:if> -->
   <!-- If the gripper bar is being used, then also add the gripper bar -->
-  <xacro:if value="$(arg show_gripper_bar)">
+  <!-- <xacro:if value="$(arg show_gripper_bar)">
     <joint name="gripper_bar" type="fixed">
       <axis xyz="1 0 0"/>
@@ -383,7 +383,7 @@
         <inertia ixx="0.001" iyy="0.001" izz="0.001" ixy="0" ixz="0" iyz="0" />
       </inertial>
-    </link>
+    </link> -->
     <!-- If the gripper fingers are being used, add those as well -->
-    <xacro:if value="$(arg show_gripper_fingers)">
+    <!-- <xacro:if value="$(arg show_gripper_fingers)">
       <joint name="left_finger" type="prismatic">
         <axis xyz="0 1 0"/>
@@ -476,5 +476,5 @@
       </link>
     </xacro:if>
-  </xacro:if>
+  </xacro:if> -->
   <xacro:if value="${urdf_loc != ''}">
     <xacro:include filename="${urdf_loc}"/>

File: interbotix_ros_xsarms/interbotix_xsarm_moveit/config/srdf/mobile_wx250s.srdf.xacro (robot description, xacro)
@@ -23,12 +23,12 @@
         <joint name="wrist_rotate" />
         <joint name="ee_arm" />
-        <joint name="gripper_bar" />
+        <!-- <joint name="gripper_bar" />
         <joint name="ee_bar" />
-        <joint name="ee_gripper" />
+        <joint name="ee_gripper" /> -->
     </group>
-    <group name="interbotix_gripper">
+    <!-- <group name="interbotix_gripper">
         <link name="$(arg robot_name)/left_finger_link" />
         <link name="$(arg robot_name)/right_finger_link" />
-    </group>
+    </group> -->
     <!--GROUP STATES: Purpose: Define a named state for a particular group, in terms of joint values. This is useful to define states like 'folded arms'-->
     <group_state name="Home" group="interbotix_arm">
@@ -49,12 +49,12 @@
     </group_state>
     <group_state name="Sleep" group="interbotix_arm">
-        <joint name="elbow" value="1.55" />
+        <joint name="elbow" value="1.57" />
         <joint name="forearm_roll" value="0" />
-        <joint name="shoulder" value="-1.8" />
+        <joint name="shoulder" value="-1.57" />
         <joint name="waist" value="0" />
-        <joint name="wrist_angle" value="0.8" />
+        <joint name="wrist_angle" value="0" />
         <joint name="wrist_rotate" value="0" />
     </group_state>
-    <group_state name="Closed" group="interbotix_gripper">
+    <!-- <group_state name="Closed" group="interbotix_gripper">
         <joint name="left_finger" value="0.015" />
         <joint name="right_finger" value="-0.015" />
@@ -67,7 +67,7 @@
         <joint name="left_finger" value="0.0195" />
         <joint name="right_finger" value="-0.0195" />
-    </group_state>
+    </group_state> -->
     <!--END EFFECTOR: Purpose: Represent information about an end effector.-->
-    <end_effector name="interbotix_gripper" parent_link="$(arg robot_name)/ee_gripper_link" group="interbotix_gripper" />
+    <!-- <end_effector name="interbotix_gripper" parent_link="$(arg robot_name)/ee_gripper_link" group="interbotix_gripper" /> -->
     <!--DISABLE COLLISIONS: By default it is assumed that any link of the robot could potentially come into collision with any other link in the robot. This tag disables collision checking between a specified pair of links. -->
     <disable_collisions link1="$(arg robot_name)/$(arg base_link_frame)" link2="$(arg robot_name)/shoulder_link" reason="Adjacent" />
